File: Treadstone32.kicad_pcb (KiCad board)
At the start: 2 copper layers, 198.8 x 75.8 mm, 82 parts, among them SW1 SW_DIP_x01, SW10 SW_PUSH, SW11 SW_PUSH, SW12 SW_PUSH, SW13 SW_PUSH, SW14 SW_PUSH, SW15 SW_PUSH, SW16 SW_PUSH, SW17 SW_PUSH, SW18 SW_PUSH, SW19 SW_PUSH, SW2 SW_PUSH, SW20 SW_PUSH, SW21 SW_PUSH, SW22 SW_PUSH, SW23 SW_PUSH, SW24 SW_PUSH, SW25 SW_PUSH, SW26 SW_PUSH, SW27 SW_PUSH, SW28 SW_PUSH, SW29 SW_PUSH, SW3 SW_PUSH, SW30 SW_PUSH, SW31 SW_PUSH, SW32 SW_PUSH, SW33 SW_PUSH, SW4 SW_PUSH, SW5 SW_PUSH, SW6 SW_PUSH, SW7 SW_PUSH, SW8 SW_PUSH, SW9 SW_PUSH, U1 ATmega32U4-AU, X1 16MHz

Commit message: Pcb edits
Parts:
- added D33: SR05.TCT, SR05:Semtech-SOT-143-0-0-MFG, F.Cu at (200.7, 71.4)
- added R7: 1M, Resistor_SMD:R_0805_2012Metric, F.Cu at (206.9, 69.4)
- moved F1 13.0 mm to (194.4, 75.4)
- moved R2 6.00 mm to (199.2, 76.7)
- moved R3 6.00 mm to (201.8, 76.7)
Routing:
- net VBUS: track 13.0 -> 25.8 mm, vias 0 -> 2
- net D+: track 6.66 -> 15.2 mm
- net GND: track 197.5 -> 190.7 mm, vias 19 -> 20
- net D-: track 8.14 -> 14.0 mm
- net Net-(R2-Pad1): track 45.3 -> 40.2 mm
- net Net-(R7-Pad1): track 17.0 -> 21.9 mm
- net Net-(R3-Pad1): track 44.9 -> 40.3 mm
- net +5V: track 135.7 -> 138.0 mm
Other:
- board text added: "Treadstone32 revC.1 Designed by marksard 2019 Revised by Melinda 2021"
- board text removed: "Treadstone32 rev1.1 Designed by marksard 2019"
