File: Treadstone32.kicad_pcb (KiCad board)
At the start: 2 copper layers, 198.8 x 75.8 mm, 92 parts, among them SW1 SW_DIP_x01, SW10 SW_PUSH, SW11 SW_PUSH, SW12 SW_PUSH, SW13 SW_PUSH, SW14 SW_PUSH, SW15 SW_PUSH, SW16 SW_PUSH, SW17 SW_PUSH, SW18 SW_PUSH, SW19 SW_PUSH, SW2 SW_PUSH, SW20 SW_PUSH, SW21 SW_PUSH, SW22 SW_PUSH, SW23 SW_PUSH, SW24 SW_PUSH, SW25 SW_PUSH, SW26 SW_PUSH, SW27 SW_PUSH, SW28 SW_PUSH, SW29 SW_PUSH, SW3 SW_PUSH, SW30 SW_PUSH, SW31 SW_PUSH, SW32 SW_PUSH, SW33 SW_PUSH, SW4 SW_PUSH, SW5 SW_PUSH, SW6 SW_PUSH, SW7 SW_PUSH, SW8 SW_PUSH, SW9 SW_PUSH, U1 ATmega32U4-AU, X1 16MHz

Commit message: Updates
Parts:
- D1, D10, D11, D12, D13, D14, D15, D16, D17, D18, D19, D2, D20, D21, D22, D23, D24, D25, D26, D27, D28, D29, D3, D30, D31, D32, D4, D5, D6, D7, D8, D9: footprint Diode_SMD:D_0805_2012Metric -> Diode_SMD:D_SOD-123
- moved D21 2.86 mm to (102.6, 107.2)
- moved D24 2.41 mm to (164.1, 107.2)
- moved D30 2.41 mm to (283.8, 107.2)
- moved D23 2.40 mm to (145.1, 107.2)
- moved D22 2.40 mm to (126.1, 107.2)
- moved D29 2.29 mm to (268.9, 107.2)
- moved D20 2.26 mm to (283.2, 88.9)
- moved D28 2.24 mm to (249.9, 107.2)
- moved D27 2.20 mm to (230.8, 107.2)
- moved D19 2.19 mm to (264.1, 88.9)
- moved D18 2.16 mm to (245.1, 88.9)
- moved D26 2.16 mm to (211.8, 107.2)
- moved D17 2.09 mm to (226.0, 88.9)
- moved D1 2.09 mm to (107.0, 70.1)
- moved D11 2.07 mm to (111.7, 88.9)
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Routing:
- net row1: track 272.0 -> 194.9 mm
- net Net-(D24-Pad2): track 8.45 -> 5.58 mm
- net Net-(D23-Pad2): track 8.27 -> 5.56 mm
- net Net-(D22-Pad2): track 8.25 -> 5.55 mm
- net col1: track 114.9 -> 112.2 mm
- net Net-(D29-Pad2): track 8.20 -> 5.55 mm
- net Net-(D28-Pad2): track 8.18 -> 5.55 mm
- net Net-(D27-Pad2): track 8.16 -> 5.55 mm
- net Net-(D26-Pad2): track 8.13 -> 5.55 mm
- net Net-(D25-Pad2): track 8.10 -> 5.60 mm
- net Net-(D18-Pad2): track 8.79 -> 6.35 mm
- net Net-(D11-Pad2): track 8.49 -> 6.35 mm
- net Net-(D20-Pad2): track 8.37 -> 6.35 mm
- net row3: track 49.7 -> 47.7 mm
- net Net-(D8-Pad2): track 8.75 -> 6.78 mm
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