File: Treadstone32.sch (KiCad schematic (older format))
At the start: 82 parts, among them SW1 SW_DIP_x01, SW10 SW_PUSH, SW11 SW_PUSH, SW12 SW_PUSH, SW13 SW_PUSH, SW14 SW_PUSH, SW15 SW_PUSH, SW16 SW_PUSH, SW17 SW_PUSH, SW18 SW_PUSH, SW19 SW_PUSH, SW2 SW_PUSH, SW20 SW_PUSH, SW21 SW_PUSH, SW22 SW_PUSH, SW23 SW_PUSH, SW24 SW_PUSH, SW25 SW_PUSH, SW26 SW_PUSH, SW27 SW_PUSH, SW28 SW_PUSH, SW29 SW_PUSH, SW3 SW_PUSH, SW30 SW_PUSH, SW31 SW_PUSH, SW32 SW_PUSH, SW33 SW_PUSH, SW4 SW_PUSH, SW5 SW_PUSH, SW6 SW_PUSH, SW7 SW_PUSH, SW8 SW_PUSH, SW9 SW_PUSH, U1 ATmega32U4-AU, X1 16MHz

Commit message: Pcb edits
Parts:
- added D33: SR05.TCT, SR05:Semtech-SOT-143-0-0-MFG, symbol SR05:SR05.TCT
- added R7: 1M, Resistor_SMD:R_0805_2012Metric, symbol Device:R
- F1: footprint Fuse:Fuse_0805_2012Metric -> Fuse:Fuse_1206_3216Metric
- SW10, SW11, SW12, SW13, SW14, SW15, SW16, SW17, SW18, SW19, SW2, SW20, SW21, SW22, SW23, SW24, SW25, SW26, SW27, SW28, SW29, SW3, SW30, SW31, SW32, SW33, SW4, SW5, SW6, SW7, SW8, SW9: footprint kbd:CherryMX_Hotswap_front -> Button_Switch_Keyboard:SW_Cherry_MX_1.00u_PCB
Connections:
- net D+: now also D33.3 (2_I/O)
- net D-: now also D33.2 (1_I/O)
- net GND: now also D33.1 (ANODE), R7.2
- net VBUS: now also D33.4 (CATHODE)
- net at USB1.13 (SHIELD): now also R7.1
- no-connect marks 2 -> 1

Commit message: Add underglow and switch to solderable switches
Parts:
- added D34, D35, D36, D37, D38, D39, D40, D41: WS2812B, LED_SMD:LED_WS2812B_PLCC4_5.0x5.0mm_P3.2mm, symbol LED:WS2812B
- D33: symbol SR05:SR05.TCT -> Treadstone32-rescue:SR05.TCT-SR05
- F1: footprint Fuse:Fuse_1206_3216Metric -> Fuse:Fuse_0805_2012Metric
- SW10, SW11, SW12, SW13, SW14, SW15, SW16, SW17, SW18, SW19, SW2, SW20, SW21, SW22, SW23, SW24, SW25, SW26, SW27, SW28, SW29, SW3, SW30, SW31, SW32, SW33, SW4, SW5, SW6, SW7, SW8, SW9: footprint Button_Switch_Keyboard:SW_Cherry_MX_1.00u_PCB -> kbd:MXOnly-1U-NoLED
- U1: symbol MCU_Microchip_ATmega:ATmega32U4-AU -> Treadstone32-rescue:ATmega32U4-AU-MCU_Microchip_ATmega
- USB1: symbol typec:HRO-TYPE-C-31-M-12 -> Treadstone32-rescue:HRO-TYPE-C-31-M-12-typec
Connections:
- net +5V: now also D34.1 (VDD), D35.1 (VDD), D36.1 (VDD), D37.1 (VDD), D38.1 (VDD), D39.1 (VDD), D40.1 (VDD), D41.1 (VDD)
- net GND: now also D34.3 (VSS), D35.3 (VSS), D36.3 (VSS), D37.3 (VSS), D38.3 (VSS), D39.3 (VSS), D40.3 (VSS), D41.3 (VSS)
- net RGB: now reaches U1.12 (PB7)
- net RGB: now also D34.4 (DIN)
- new net: D34.2 (DOUT), D35.4 (DIN)
- new net: D35.2 (DOUT), D36.4 (DIN)
- new net: D36.2 (DOUT), D37.4 (DIN)
- new net: D37.2 (DOUT), D38.4 (DIN)
- new net: D38.2 (DOUT), D39.4 (DIN)
- new net: D39.2 (DOUT), D40.4 (DIN)
- new net: D40.2 (DOUT), D41.4 (DIN)
- no-connect marks 1 -> 2

Commit message: Updates
Parts:
- D1, D10, D11, D12, D13, D14, D15, D16, D17, D18, D19, D2, D20, D21, D22, D23, D24, D25, D26, D27, D28, D29, D3, D30, D31, D32, D4, D5, D6, D7, D8, D9: footprint Diode_SMD:D_0805_2012Metric -> Diode_SMD:D_SOD-123
Changed lines of the file:
@@
 F 0 "D1" V 1596 1221 50  0000 R CNN
 F 1 "D" V 1505 1221 50  0000 R CNN
-F 2 "Diode_SMD:D_0805_2012Metric" H 1550 1300 50  0001 C CNN
+F 2 "Diode_SMD:D_SOD-123" H 1550 1300 50  0001 C CNN
 F 3 "~" H 1550 1300 50  0001 C CNN
 	1    1550 1300
@@
 F 0 "D2" V 2446 1221 50  0000 R CNN
 F 1 "D" V 2355 1221 50  0000 R CNN
-F 2 "Diode_SMD:D_0805_2012Metric" H 2400 1300 50  0001 C CNN
+F 2 "Diode_SMD:D_SOD-123" H 2400 1300 50  0001 C CNN
 F 3 "~" H 2400 1300 50  0001 C CNN
 	1    2400 1300
@@
 F 0 "D3" V 3296 1221 50  0000 R CNN
 F 1 "D" V 3205 1221 50  0000 R CNN
-F 2 "Diode_SMD:D_0805_2012Metric" H 3250 1300 50  0001 C CNN
+F 2 "Diode_SMD:D_SOD-123" H 3250 1300 50  0001 C CNN
 F 3 "~" H 3250 1300 50  0001 C CNN
 	1    3250 1300
@@
 F 0 "D4" V 4146 1221 50  0000 R CNN
 F 1 "D" V 4055 1221 50  0000 R CNN
-F 2 "Diode_SMD:D_0805_2012Metric" H 4100 1300 50  0001 C CNN
+F 2 "Diode_SMD:D_SOD-123" H 4100 1300 50  0001 C CNN
 F 3 "~" H 4100 1300 50  0001 C CNN
 	1    4100 1300
@@
 F 0 "D5" V 4996 1221 50  0000 R CNN
 F 1 "D" V 4905 1221 50  0000 R CNN
-F 2 "Diode_SMD:D_0805_2012Metric" H 4950 1300 50  0001 C CNN
+F 2 "Diode_SMD:D_SOD-123" H 4950 1300 50  0001 C CNN
 F 3 "~" H 4950 1300 50  0001 C CNN
 	1    4950 1300
@@
 F 0 "D11" V 1596 1921 50  0000 R CNN
 F 1 "D" V 1505 1921 50  0000 R CNN
-F 2 "Diode_SMD:D_0805_2012Metric" H 1550 2000 50  0001 C CNN
+F 2 "Diode_SMD:D_SOD-123" H 1550 2000 50  0001 C CNN
 F 3 "~" H 1550 2000 50  0001 C CNN
 	1    1550 2000
@@
 F 0 "D12" V 2446 1921 50  0000 R CNN
 F 1 "D" V 2355 1921 50  0000 R CNN
-F 2 "Diode_SMD:D_0805_2012Metric" H 2400 2000 50  0001 C CNN
+F 2 "Diode_SMD:D_SOD-123" H 2400 2000 50  0001 C CNN
 F 3 "~" H 2400 2000 50  0001 C CNN
 	1    2400 2000
@@
 F 0 "D13" V 3296 1921 50  0000 R CNN
 F 1 "D" V 3205 1921 50  0000 R CNN
-F 2 "Diode_SMD:D_0805_2012Metric" H 3250 2000 50  0001 C CNN
+F 2 "Diode_SMD:D_SOD-123" H 3250 2000 50  0001 C CNN
 F 3 "~" H 3250 2000 50  0001 C CNN
 	1    3250 2000
@@
 F 0 "D14" V 4146 1921 50  0000 R CNN
 F 1 "D" V 4055 1921 50  0000 R CNN
-F 2 "Diode_SMD:D_0805_2012Metric" H 4100 2000 50  0001 C CNN
+F 2 "Diode_SMD:D_SOD-123" H 4100 2000 50  0001 C CNN
 F 3 "~" H 4100 2000 50  0001 C CNN
 	1    4100 2000
@@
 F 0 "D15" V 4996 1921 50  0000 R CNN
 F 1 "D" V 4905 1921 50  0000 R CNN
-F 2 "Diode_SMD:D_0805_2012Metric" H 4950 2000 50  0001 C CNN
+F 2 "Diode_SMD:D_SOD-123" H 4950 2000 50  0001 C CNN
 F 3 "~" H 4950 2000 50  0001 C CNN
 	1    4950 2000
@@
 F 0 "D21" V 1596 2621 50  0000 R CNN
 F 1 "D" V 1505 2621 50  0000 R CNN
-F 2 "Diode_SMD:D_0805_2012Metric" H 1550 2700 50  0001 C CNN
+F 2 "Diode_SMD:D_SOD-123" H 1550 2700 50  0001 C CNN
 F 3 "~" H 1550 2700 50  0001 C CNN
 	1    1550 2700
@@
 F 0 "D22" V 2446 2621 50  0000 R CNN
 F 1 "D" V 2355 2621 50  0000 R CNN
-F 2 "Diode_SMD:D_0805_2012Metric" H 2400 2700 50  0001 C CNN
+F 2 "Diode_SMD:D_SOD-123" H 2400 2700 50  0001 C CNN
 F 3 "~" H 2400 2700 50  0001 C CNN
 	1    2400 2700
@@
 F 0 "D23" V 3296 2621 50  0000 R CNN
 F 1 "D" V 3205 2621 50  0000 R CNN
-F 2 "Diode_SMD:D_0805_2012Metric" H 3250 2700 50  0001 C CNN
+F 2 "Diode_SMD:D_SOD-123" H 3250 2700 50  0001 C CNN
 F 3 "~" H 3250 2700 50  0001 C CNN
 	1    3250 2700
@@
 F 0 "D24" V 4146 2621 50  0000 R CNN
 F 1 "D" V 4055 2621 50  0000 R CNN
-F 2 "Diode_SMD:D_0805_2012Metric" H 4100 2700 50  0001 C CNN
+F 2 "Diode_SMD:D_SOD-123" H 4100 2700 50  0001 C CNN
 F 3 "~" H 4100 2700 50  0001 C CNN
 	1    4100 2700
@@
 F 0 "D25" V 4996 2621 50  0000 R CNN
 F 1 "D" V 4905 2621 50  0000 R CNN
-F 2 "Diode_SMD:D_0805_2012Metric" H 4950 2700 50  0001 C CNN
+F 2 "Diode_SMD:D_SOD-123" H 4950 2700 50  0001 C CNN
 F 3 "~" H 4950 2700 50  0001 C CNN
 	1    4950 2700
@@
 F 0 "D31" V 4996 3321 50  0000 R CNN
 F 1 "D" V 4905 3321 50  0000 R CNN
-F 2 "Diode_SMD:D_0805_2012Metric" H 4950 3400 50  0001 C CNN
+F 2 "Diode_SMD:D_SOD-123" H 4950 3400 50  0001 C CNN
 F 3 "~" H 4950 3400 50  0001 C CNN
 	1    4950 3400
@@
 F 0 "D6" V 5966 1221 50  0000 R CNN
 F 1 "D" V 5875 1221 50  0000 R CNN
-F 2 "Diode_SMD:D_0805_2012Metric" H 5920 1300 50  0001 C CNN
+F 2 "Diode_SMD:D_SOD-123" H 5920 1300 50  0001 C CNN
 F 3 "~" H 5920 1300 50  0001 C CNN
 	1    5920 1300
@@
 F 0 "D7" V 6816 1221 50  0000 R CNN
 F 1 "D" V 6725 1221 50  0000 R CNN
-F 2 "Diode_SMD:D_0805_2012Metric" H 6770 1300 50  0001 C CNN
+F 2 "Diode_SMD:D_SOD-123" H 6770 1300 50  0001 C CNN
 F 3 "~" H 6770 1300 50  0001 C CNN
 	1    6770 1300
@@
 F 0 "D8" V 7666 1221 50  0000 R CNN
 F 1 "D" V 7575 1221 50  0000 R CNN
-F 2 "Diode_SMD:D_0805_2012Metric" H 7620 1300 50  0001 C CNN
+F 2 "Diode_SMD:D_SOD-123" H 7620 1300 50  0001 C CNN
 F 3 "~" H 7620 1300 50  0001 C CNN
 	1    7620 1300
@@
 F 0 "D9" V 8516 1221 50  0000 R CNN
 F 1 "D" V 8425 1221 50  0000 R CNN
-F 2 "Diode_SMD:D_0805_2012Metric" H 8470 1300 50  0001 C CNN
+F 2 "Diode_SMD:D_SOD-123" H 8470 1300 50  0001 C CNN
 F 3 "~" H 8470 1300 50  0001 C CNN
 	1    8470 1300
@@
 F 0 "D10" V 9366 1221 50  0000 R CNN
 F 1 "D" V 9275 1221 50  0000 R CNN
-F 2 "Diode_SMD:D_0805_2012Metric" H 9320 1300 50  0001 C CNN
+F 2 "Diode_SMD:D_SOD-123" H 9320 1300 50  0001 C CNN
 F 3 "~" H 9320 1300 50  0001 C CNN
 	1    9320 1300
@@
 F 0 "D16" V 5966 1921 50  0000 R CNN
 F 1 "D" V 5875 1921 50  0000 R CNN
-F 2 "Diode_SMD:D_0805_2012Metric" H 5920 2000 50  0001 C CNN
+F 2 "Diode_SMD:D_SOD-123" H 5920 2000 50  0001 C CNN
 F 3 "~" H 5920 2000 50  0001 C CNN
 	1    5920 2000
@@
 F 0 "D17" V 6816 1921 50  0000 R CNN
 F 1 "D" V 6725 1921 50  0000 R CNN
-F 2 "Diode_SMD:D_0805_2012Metric" H 6770 2000 50  0001 C CNN
+F 2 "Diode_SMD:D_SOD-123" H 6770 2000 50  0001 C CNN
 F 3 "~" H 6770 2000 50  0001 C CNN
 	1    6770 2000
@@
 F 0 "D18" V 7666 1921 50  0000 R CNN
 F 1 "D" V 7575 1921 50  0000 R CNN
-F 2 "Diode_SMD:D_0805_2012Metric" H 7620 2000 50  0001 C CNN
+F 2 "Diode_SMD:D_SOD-123" H 7620 2000 50  0001 C CNN
 F 3 "~" H 7620 2000 50  0001 C CNN
 	1    7620 2000
@@
 F 0 "D19" V 8516 1921 50  0000 R CNN
 F 1 "D" V 8425 1921 50  0000 R CNN
-F 2 "Diode_SMD:D_0805_2012Metric" H 8470 2000 50  0001 C CNN
+F 2 "Diode_SMD:D_SOD-123" H 8470 2000 50  0001 C CNN
 F 3 "~" H 8470 2000 50  0001 C CNN
 	1    8470 2000
@@
 F 0 "D20" V 9366 1921 50  0000 R CNN
 F 1 "D" V 9275 1921 50  0000 R CNN
-F 2 "Diode_SMD:D_0805_2012Metric" H 9320 2000 50  0001 C CNN
+F 2 "Diode_SMD:D_SOD-123" H 9320 2000 50  0001 C CNN
 F 3 "~" H 9320 2000 50  0001 C CNN
 	1    9320 2000
@@
 F 0 "D26" V 5966 2621 50  0000 R CNN
 F 1 "D" V 5875 2621 50  0000 R CNN
-F 2 "Diode_SMD:D_0805_2012Metric" H 5920 2700 50  0001 C CNN
+F 2 "Diode_SMD:D_SOD-123" H 5920 2700 50  0001 C CNN
 F 3 "~" H 5920 2700 50  0001 C CNN
 	1    5920 2700
@@
 F 0 "D27" V 6816 2621 50  0000 R CNN
 F 1 "D" V 6725 2621 50  0000 R CNN
-F 2 "Diode_SMD:D_0805_2012Metric" H 6770 2700 50  0001 C CNN
+F 2 "Diode_SMD:D_SOD-123" H 6770 2700 50  0001 C CNN
 F 3 "~" H 6770 2700 50  0001 C CNN
 	1    6770 2700
@@
 F 0 "D28" V 7666 2621 50  0000 R CNN
 F 1 "D" V 7575 2621 50  0000 R CNN
-F 2 "Diode_SMD:D_0805_2012Metric" H 7620 2700 50  0001 C CNN
+F 2 "Diode_SMD:D_SOD-123" H 7620 2700 50  0001 C CNN
 F 3 "~" H 7620 2700 50  0001 C CNN
 	1    7620 2700
@@
 F 0 "D29" V 8516 2621 50  0000 R CNN
 F 1 "D" V 8425 2621 50  0000 R CNN
-F 2 "Diode_SMD:D_0805_2012Metric" H 8470 2700 50  0001 C CNN
+F 2 "Diode_SMD:D_SOD-123" H 8470 2700 50  0001 C CNN
 F 3 "~" H 8470 2700 50  0001 C CNN
 	1    8470 2700
@@
 F 0 "D30" V 9366 2621 50  0000 R CNN
 F 1 "D" V 9275 2621 50  0000 R CNN
-F 2 "Diode_SMD:D_0805_2012Metric" H 9320 2700 50  0001 C CNN
+F 2 "Diode_SMD:D_SOD-123" H 9320 2700 50  0001 C CNN
 F 3 "~" H 9320 2700 50  0001 C CNN
 	1    9320 2700
@@
 F 0 "D32" V 5966 3321 50  0000 R CNN
 F 1 "D" V 5875 3321 50  0000 R CNN
-F 2 "Diode_SMD:D_0805_2012Metric" H 5920 3400 50  0001 C CNN
+F 2 "Diode_SMD:D_SOD-123" H 5920 3400 50  0001 C CNN
 F 3 "~" H 5920 3400 50  0001 C CNN
 	1    5920 3400
